File: circuit/misc.sch (KiCad schematic (older format))
At the start: 1 part

Commit message: Add resistor on misc
Parts:
- removed D?: LED_Cree_XHP50_12V, LEDs:LED_CREE-XHP50_12V, symbol LED:LED_Cree_XHP50_12V
- added R?: R, symbol pspice:R
Changed lines of the file:
@@
 $EndDescr
 $Comp
-L LED:LED_Cree_XHP50_12V D?
-U 1 1 5A75F301
-P 6000 3150
-F 0 "D?" H 6000 3430 50  0000 C CNN
-F 1 "LED_Cree_XHP50_12V" H 6000 3339 50  0000 C CNN
-F 2 "LEDs:LED_CREE-XHP50_12V" H 6000 3475 50  0001 C CNN
-F 3 "http://www.cree.com/%7E/media/Files/Cree/LED%20Components%20and%20Modules/XLamp/Data%20and%20Binning/ds%20XHP50.pdf" H 5800 3150 50  0001 C CNN
-	1    6000 3150
+L pspice:R R?
+U 1 1 5A75F33D
+P 6000 3850
+F 0 "R?" H 6068 3896 50  0000 L CNN
+F 1 "R" H 6068 3805 50  0000 L CNN
+F 2 "" H 6000 3850 50  0001 C CNN
+F 3 "" H 6000 3850 50  0001 C CNN
+	1    6000 3850
 	1    0    0    -1
 $EndComp

Commit message: last changes
Parts:
- added R? (x2): R, symbol pspice:R
Changed lines of the file:
@@
+	1    0    0    -1
+$EndComp
+$Comp
+L pspice:R R?
+U 1 1 5A75F36F
+P 6250 3850
+F 0 "R?" H 6318 3896 50  0000 L CNN
+F 1 "R" H 6318 3805 50  0000 L CNN
+F 2 "" H 6250 3850 50  0001 C CNN
+F 3 "" H 6250 3850 50  0001 C CNN
+	1    6250 3850
+	1    0    0    -1
+$EndComp
+$Comp
+L pspice:R R?
+U 1 1 5A75F386
+P 6500 3850
+F 0 "R?" H 6568 3896 50  0000 L CNN
+F 1 "R" H 6568 3805 50  0000 L CNN
+F 2 "" H 6500 3850 50  0001 C CNN
+F 3 "" H 6500 3850 50  0001 C CNN
+	1    6500 3850
 	1    0    0    -1
 $EndComp
